File: matrix.sch (KiCad schematic (older format))
At the start: 128 parts

Commit message: new switches are now in PCB file
Parts:
- D_R0C0, D_R0C1, D_R0C10, D_R0C11, D_R0C12, D_R0C13, D_R0C14, D_R0C15, D_R0C2, D_R0C3, D_R0C4, D_R0C5, D_R0C6, D_R0C7, D_R0C8, D_R0C9, D_R1C0, D_R1C1, D_R1C10, D_R1C11, D_R1C12, D_R1C13, D_R1C14, D_R1C15, D_R1C2, D_R1C3, D_R1C4, D_R1C5, D_R1C6, D_R1C7, D_R1C8, D_R1C9, D_R2C0, D_R2C1, D_R2C10, D_R2C11, D_R2C12, D_R2C13, D_R2C14, D_R2C15, D_R2C2, D_R2C3, D_R2C4, D_R2C5, D_R2C6, D_R2C7, D_R2C8, D_R2C9, D_R3C0, D_R3C1, D_R3C10, D_R3C11, D_R3C12, D_R3C13, D_R3C14, D_R3C15, D_R3C2, D_R3C3, D_R3C4, D_R3C5, D_R3C6, D_R3C7, D_R3C8, D_R3C9: footprint (none) -> Diode_SMD:D_SOD-123
- MX_R0C0_ESC1: renamed from MX_R0C0_ESC; footprint (none) -> MX_Alps_Hybrid:MX-1U-NoLED
- MX_R0C10_P1: renamed from MX_R0C10_P; footprint (none) -> MX_Alps_Hybrid:MX-1U-NoLED
- MX_R0C11_LBRKT1: renamed from MX_R0C11_LBRKT; footprint (none) -> MX_Alps_Hybrid:MX-1U-NoLED
- MX_R0C12_RBRKT1: renamed from MX_R0C12_RBRKT; footprint (none) -> MX_Alps_Hybrid:MX-1U-NoLED
- MX_R0C13_7, MX_R0C14_8, MX_R0C15_9, MX_R1C13_4, MX_R1C14_5, MX_R1C15_6, MX_R2C13_1, MX_R2C14_2, MX_R2C15_3, MX_R3C13_0: footprint (none) -> MX_Alps_Hybrid:MX-1U-NoLED
- MX_R0C1_Q1: renamed from MX_R0C1_Q; footprint (none) -> MX_Alps_Hybrid:MX-1U-NoLED
- MX_R0C2_W1: renamed from MX_R0C2_W; footprint (none) -> MX_Alps_Hybrid:MX-1U-NoLED
- MX_R0C3_E1: renamed from MX_R0C3_E; footprint (none) -> MX_Alps_Hybrid:MX-1U-NoLED
- MX_R0C4_R1: renamed from MX_R0C4_R; footprint (none) -> MX_Alps_Hybrid:MX-1U-NoLED
- MX_R0C5_T1: renamed from MX_R0C5_T; footprint (none) -> MX_Alps_Hybrid:MX-1U-NoLED
- MX_R0C6_Y1: renamed from MX_R0C6_Y; footprint (none) -> MX_Alps_Hybrid:MX-1U-NoLED
- MX_R0C7_U1: renamed from MX_R0C7_U; footprint (none) -> MX_Alps_Hybrid:MX-1U-NoLED
- MX_R0C8_I1: renamed from MX_R0C8_I; footprint (none) -> MX_Alps_Hybrid:MX-1U-NoLED
- MX_R0C9_O1: renamed from MX_R0C9_O; footprint (none) -> MX_Alps_Hybrid:MX-1U-NoLED
- MX_R1C0_TAB1: renamed from MX_R1C0_TAB; footprint (none) -> MX_Alps_Hybrid:MX-1U-NoLED
- MX_R1C10_SCLN1: renamed from MX_R1C10_SCLN; footprint (none) -> MX_Alps_Hybrid:MX-1U-NoLED
- MX_R1C11_SQTE1: renamed from MX_R1C11_SQTE; footprint (none) -> MX_Alps_Hybrid:MX-1U-NoLED
- MX_R1C12_RTRN1: renamed from MX_R1C12_RTRN; footprint (none) -> MX_Alps_Hybrid:MX-1U-NoLED
- MX_R1C1_A1: renamed from MX_R1C1_A; footprint (none) -> MX_Alps_Hybrid:MX-1U-NoLED
- MX_R1C2_S1: renamed from MX_R1C2_S; footprint (none) -> MX_Alps_Hybrid:MX-1U-NoLED
- MX_R1C3_D1: renamed from MX_R1C3_D; footprint (none) -> MX_Alps_Hybrid:MX-1U-NoLED
- MX_R1C4_F1: renamed from MX_R1C4_F; footprint (none) -> MX_Alps_Hybrid:MX-1U-NoLED
- MX_R1C5_G1: renamed from MX_R1C5_G; footprint (none) -> MX_Alps_Hybrid:MX-1U-NoLED
- MX_R1C6_H1: renamed from MX_R1C6_H; footprint (none) -> MX_Alps_Hybrid:MX-1U-NoLED
- MX_R1C7_J1: renamed from MX_R1C7_J; footprint (none) -> MX_Alps_Hybrid:MX-1U-NoLED
- MX_R1C8_K1: renamed from MX_R1C8_K; footprint (none) -> MX_Alps_Hybrid:MX-1U-NoLED
- MX_R1C9_L1: renamed from MX_R1C9_L; footprint (none) -> MX_Alps_Hybrid:MX-1U-NoLED
- MX_R2C0_SHIFT1: renamed from MX_R2C0_SHIFT; footprint (none) -> MX_Alps_Hybrid:MX-1U-NoLED
- MX_R2C10_SLSH1: renamed from MX_R2C10_SLSH; footprint (none) -> MX_Alps_Hybrid:MX-1U-NoLED
- MX_R2C11_BSLSH1: renamed from MX_R2C11_BSLSH; footprint (none) -> MX_Alps_Hybrid:MX-1U-NoLED
- MX_R2C12_UARR1: renamed from MX_R2C12_UARR; footprint (none) -> MX_Alps_Hybrid:MX-1U-NoLED
- MX_R2C1_Z1: renamed from MX_R2C1_Z; footprint (none) -> MX_Alps_Hybrid:MX-1U-NoLED
- MX_R2C3_C1: renamed from MX_R2C3_C; footprint (none) -> MX_Alps_Hybrid:MX-1U-NoLED
- MX_R2C4_V1: renamed from MX_R2C4_V; footprint (none) -> MX_Alps_Hybrid:MX-1U-NoLED
- MX_R2C5_B1: renamed from MX_R2C5_B; footprint (none) -> MX_Alps_Hybrid:MX-1U-NoLED
- MX_R2C6_N1: renamed from MX_R2C6_N; footprint (none) -> MX_Alps_Hybrid:MX-1U-NoLED
- MX_R2C7_M1: renamed from MX_R2C7_M; footprint (none) -> MX_Alps_Hybrid:MX-1U-NoLED
- MX_R2C8_CMMA1: renamed from MX_R2C8_CMMA; footprint (none) -> MX_Alps_Hybrid:MX-1U-NoLED
- MX_R2C9_PERI1: renamed from MX_R2C9_PERI; footprint (none) -> MX_Alps_Hybrid:MX-1U-NoLED
- MX_R3C0_FN1: renamed from MX_R3C0_FN; footprint (none) -> MX_Alps_Hybrid:MX-1U-NoLED
- MX_R3C10_RSHIFT1: renamed from MX_R3C10_RSHIFT; footprint (none) -> MX_Alps_Hybrid:MX-1U-NoLED
- MX_R3C11_LARR1: renamed from MX_R3C11_LARR; footprint (none) -> MX_Alps_Hybrid:MX-1U-NoLED
- MX_R3C12_DARR1: renamed from MX_R3C12_DARR; footprint (none) -> MX_Alps_Hybrid:MX-1U-NoLED
- MX_R3C13_RARR1: renamed from MX_R3C13_RARR; footprint (none) -> MX_Alps_Hybrid:MX-1U-NoLED
- MX_R3C15_BKSPC1: renamed from MX_R3C15_BKSPC; footprint (none) -> MX_Alps_Hybrid:MX-1U-NoLED
- MX_R3C1_CTRLL1: renamed from MX_R3C1_CTRLL; footprint (none) -> MX_Alps_Hybrid:MX-1U-NoLED
- MX_R3C2_ALTL1: renamed from MX_R3C2_ALTL; footprint (none) -> MX_Alps_Hybrid:MX-1U-NoLED
- MX_R3C2_X1: renamed from MX_R3C2_X; footprint (none) -> MX_Alps_Hybrid:MX-1U-NoLED
- MX_R3C3_CMDL1: renamed from MX_R3C3_CMDL; footprint (none) -> MX_Alps_Hybrid:MX-1U-NoLED
- MX_R3C4_LAYRD1: renamed from MX_R3C4_LAYRD; footprint (none) -> MX_Alps_Hybrid:MX-1U-NoLED
- MX_R3C5_SPCEL1: renamed from MX_R3C5_SPCEL; footprint (none) -> MX_Alps_Hybrid:MX-1U-NoLED
- MX_R3C6_SPCER1: renamed from MX_R3C6_SPCER; footprint (none) -> MX_Alps_Hybrid:MX-1U-NoLED
- MX_R3C7_LYERU1: renamed from MX_R3C7_LYERU; footprint (none) -> MX_Alps_Hybrid:MX-1U-NoLED
- MX_R3C8_CMDR1: renamed from MX_R3C8_CMDR; footprint (none) -> MX_Alps_Hybrid:MX-1U-NoLED
- MX_R3C9_ALTR1: renamed from MX_R3C9_ALTR; footprint (none) -> MX_Alps_Hybrid:MX-1U-NoLED

Commit message: I just wired up a 63-key board. yiiikes.
Parts:
- renumbered MX_R0C15_9 to MX_R0C15_BKSPC1, MX_R1C15_6 to MX_R1C15_9, MX_R2C15_3 to MX_R2C15_6, MX_R3C2_X1 to MX_R2C2_X1, MX_R3C13_0 to MX_R3C14_0, MX_R3C15_BKSPC1 to MX_R3C15_1
Changed lines of the file:
@@
 $EndComp
 $Comp
-L MX_Alps_Hybrid:MX-NoLED MX_R3C15_BKSPC1
+L MX_Alps_Hybrid:MX-NoLED MX_R3C15_1
 U 1 1 5F6D5FCE
 P 10950 4700
-F 0 "MX_R3C15_BKSPC1" H 10983 4917 52  0000 C CNN
+F 0 "MX_R3C15_1" H 10983 4917 52  0000 C CNN
 F 1 "MX-NoLED" H 10983 4849 20  0000 C CNN
 F 2 "MX_Alps_Hybrid:MX-1U-NoLED" H 10325 4675 60  0001 C CNN
@@
 $EndComp
 $Comp
-L MX_Alps_Hybrid:MX-NoLED MX_R2C15_3
+L MX_Alps_Hybrid:MX-NoLED MX_R2C15_6
 U 1 1 5F6D5FC1
 P 10950 4000
-F 0 "MX_R2C15_3" H 10983 4217 52  0000 C CNN
+F 0 "MX_R2C15_6" H 10983 4217 52  0000 C CNN
 F 1 "MX-NoLED" H 10983 4149 20  0000 C CNN
 F 2 "MX_Alps_Hybrid:MX-1U-NoLED" H 10325 3975 60  0001 C CNN
@@
 $EndComp
 $Comp
-L MX_Alps_Hybrid:MX-NoLED MX_R1C15_6
+L MX_Alps_Hybrid:MX-NoLED MX_R1C15_9
 U 1 1 5F6D5FB4
 P 10950 3300
-F 0 "MX_R1C15_6" H 10983 3517 52  0000 C CNN
+F 0 "MX_R1C15_9" H 10983 3517 52  0000 C CNN
 F 1 "MX-NoLED" H 10983 3449 20  0000 C CNN
 F 2 "MX_Alps_Hybrid:MX-1U-NoLED" H 10325 3275 60  0001 C CNN
@@
 $EndComp
 $Comp
-L MX_Alps_Hybrid:MX-NoLED MX_R0C15_9
+L MX_Alps_Hybrid:MX-NoLED MX_R0C15_BKSPC1
 U 1 1 5F6D5FA7
 P 10950 2600
-F 0 "MX_R0C15_9" H 10983 2817 52  0000 C CNN
+F 0 "MX_R0C15_BKSPC1" H 10983 2817 52  0000 C CNN
 F 1 "MX-NoLED" H 10983 2749 20  0000 C CNN
 F 2 "MX_Alps_Hybrid:MX-1U-NoLED" H 10325 2575 60  0001 C CNN
@@
 $EndComp
 $Comp
-L MX_Alps_Hybrid:MX-NoLED MX_R3C13_0
+L MX_Alps_Hybrid:MX-NoLED MX_R3C14_0
 U 1 1 5F6D5F9A
 P 10300 4700
-F 0 "MX_R3C13_0" H 10333 4917 52  0000 C CNN
+F 0 "MX_R3C14_0" H 10333 4917 52  0000 C CNN
 F 1 "MX-NoLED" H 10333 4849 20  0000 C CNN
 F 2 "MX_Alps_Hybrid:MX-1U-NoLED" H 9675 4675 60  0001 C CNN
@@
 $EndComp
 $Comp
-L MX_Alps_Hybrid:MX-NoLED MX_R3C2_X1
+L MX_Alps_Hybrid:MX-NoLED MX_R2C2_X1
 U 1 1 5F61B68B
 P 2550 4000
-F 0 "MX_R3C2_X1" H 2583 4217 52  0000 C CNN
+F 0 "MX_R2C2_X1" H 2583 4217 52  0000 C CNN
 F 1 "MX-NoLED" H 2583 4149 20  0000 C CNN
 F 2 "MX_Alps_Hybrid:MX-1U-NoLED" H 1925 3975 60  0001 C CNN

Commit message: a few extra tweeks including silkscreen color and adding ground fill
Parts:
- MX_R0C15_BKSPC1, MX_R3C14_0: value MX-NoLED -> MX-2U-NoLED; footprint MX_Alps_Hybrid:MX-1U-NoLED -> MX_Alps_Hybrid:MX-2U-NoLED
Changed lines of the file:
@@
 P 10950 2600
 F 0 "MX_R0C15_BKSPC1" H 10983 2817 52  0000 C CNN
-F 1 "MX-NoLED" H 10983 2749 20  0000 C CNN
-F 2 "MX_Alps_Hybrid:MX-1U-NoLED" H 10325 2575 60  0001 C CNN
+F 1 "MX-2U-NoLED" H 10983 2749 20  0000 C CNN
+F 2 "MX_Alps_Hybrid:MX-2U-NoLED" H 10325 2575 60  0001 C CNN
 F 3 "" H 10325 2575 60  0001 C CNN
 	1    10950 2600
@@
 P 10300 4700
 F 0 "MX_R3C14_0" H 10333 4917 52  0000 C CNN
-F 1 "MX-NoLED" H 10333 4849 20  0000 C CNN
-F 2 "MX_Alps_Hybrid:MX-1U-NoLED" H 9675 4675 60  0001 C CNN
+F 1 "MX-2U-NoLED" H 10333 4849 20  0000 C CNN
+F 2 "MX_Alps_Hybrid:MX-2U-NoLED" H 9675 4675 60  0001 C CNN
 F 3 "" H 9675 4675 60  0001 C CNN
 	1    10300 4700
