File: keybored.kicad_pcb (KiCad board)
At the start: 2 copper layers, 24 parts, among them SW1 SW_Push, U1 ATmega32U4-AU, Y1 16MHz

Commit message: first render
Routing:
- added copper zone on B.Cu, net GND
Other:
- board text added: "KeyBored"
Changed lines of the file:
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@@
   (general
     (thickness 1.6)
-    (drawings 11)
+    (drawings 12)
     (tracks 212)
     (zones 0)
@@
       (rotate (xyz 0 0 0))
     )
+  )
+  (gr_text KeyBored (at 56.515 115.697) (layer F.SilkS)
+    (effects (font (size 1 1) (thickness 0.15)))
   )
   (gr_line (start 42.06875 79.375) (end 57.94375 79.375) (layer F.SilkS) (width 0.12))
@@
   (segment (start 79.296 109.31475) (end 79.375 109.39375) (width 0.254) (layer B.Cu) (net 20))
   (segment (start 76.3755 109.31475) (end 79.296 109.31475) (width 0.254) (layer B.Cu) (net 20))
+  (zone (net 2) (net_name GND) (layer B.Cu) (hatch edge 0.508)
+    (connect_pads (clearance 0.508))
+    (min_thickness 0.254)
+    (fill yes (arc_segments 32) (thermal_gap 0.508) (thermal_bridge_width 0.508))
+    (polygon
+      (pts
+        (xy 79.883 80.264) (xy 41.021 80.137) (xy 41.021 116.713) (xy 42.164 117.221) (xy 80.772 117.094)
+        (xy 80.391 80.137)
+      )
+    )
+  )
 )

Commit message: new switches are now in PCB file
Parts:
- removed D1, D2, D3, D4: SOD-123, Diode_SMD:D_SOD-123
- removed MX1, MX2, MX3, MX4: MX-NoLED, MX_Alps_Hybrid:MX-1U
- added D_R0C0: Diode, Diode_SMD:D_SOD-123, F.Cu at (136.3, 141.2)
- added D_R0C1: Diode, Diode_SMD:D_SOD-123, F.Cu at (142.0, 137.9)
- added D_R0C10: Diode, Diode_SMD:D_SOD-123, F.Cu at (107.5, 147.9)
- added D_R0C11: Diode, Diode_SMD:D_SOD-123, F.Cu at (101.8, 147.9)
- added D_R0C12: Diode, Diode_SMD:D_SOD-123, F.Cu at (113.3, 144.6)
- added D_R0C13: Diode, Diode_SMD:D_SOD-123, F.Cu at (107.5, 144.6)
- added D_R0C14: Diode, Diode_SMD:D_SOD-123, F.Cu at (101.8, 144.6)
- added D_R0C15: Diode, Diode_SMD:D_SOD-123, F.Cu at (119.0, 141.2)
- added D_R0C2: Diode, Diode_SMD:D_SOD-123, F.Cu at (136.3, 137.9)
- added D_R0C3: Diode, Diode_SMD:D_SOD-123, F.Cu at (130.5, 141.2)
- added D_R0C4: Diode, Diode_SMD:D_SOD-123, F.Cu at (124.8, 144.6)
- added D_R0C5: Diode, Diode_SMD:D_SOD-123, F.Cu at (119.0, 147.9)
- added D_R0C6: Diode, Diode_SMD:D_SOD-123, F.Cu at (124.8, 141.2)
- added D_R0C7: Diode, Diode_SMD:D_SOD-123, F.Cu at (119.0, 144.6)
- added D_R0C8: Diode, Diode_SMD:D_SOD-123, F.Cu at (130.5, 137.9)
- added D_R0C9: Diode, Diode_SMD:D_SOD-123, F.Cu at (113.3, 147.9)
- added D_R1C0: Diode, Diode_SMD:D_SOD-123, F.Cu at (113.3, 141.2)
- added D_R1C1: Diode, Diode_SMD:D_SOD-123, F.Cu at (124.8, 137.9)
- added D_R1C10: Diode, Diode_SMD:D_SOD-123, F.Cu at (96.0, 144.6)
- added D_R1C11: Diode, Diode_SMD:D_SOD-123, F.Cu at (90.3, 144.6)
- added D_R1C12: Diode, Diode_SMD:D_SOD-123, F.Cu at (96.0, 141.2)
- added D_R1C13: Diode, Diode_SMD:D_SOD-123, F.Cu at (101.8, 137.9)
- added D_R1C14: Diode, Diode_SMD:D_SOD-123, F.Cu at (96.0, 137.9)
- added D_R1C15: Diode, Diode_SMD:D_SOD-123, F.Cu at (90.3, 141.2)
- added D_R1C2: Diode, Diode_SMD:D_SOD-123, F.Cu at (119.0, 137.9)
- added D_R1C3: Diode, Diode_SMD:D_SOD-123, F.Cu at (113.3, 137.9)
- added D_R1C4: Diode, Diode_SMD:D_SOD-123, F.Cu at (107.5, 141.2)
- added D_R1C5: Diode, Diode_SMD:D_SOD-123, F.Cu at (101.8, 141.2)
- added D_R1C6: Diode, Diode_SMD:D_SOD-123, F.Cu at (96.0, 147.9)
- added D_R1C7: Diode, Diode_SMD:D_SOD-123, F.Cu at (107.5, 137.9)
- added D_R1C8: Diode, Diode_SMD:D_SOD-123, F.Cu at (90.3, 147.9)
- added D_R1C9: Diode, Diode_SMD:D_SOD-123, F.Cu at (84.5, 147.9)
- added D_R2C0: Diode, Diode_SMD:D_SOD-123, F.Cu at (84.5, 144.6)
- added D_R2C1: Diode, Diode_SMD:D_SOD-123, F.Cu at (78.8, 147.9)
- added D_R2C10: Diode, Diode_SMD:D_SOD-123, F.Cu at (61.5, 144.6)
- added D_R2C11: Diode, Diode_SMD:D_SOD-123, F.Cu at (78.8, 141.2)
- added D_R2C12: Diode, Diode_SMD:D_SOD-123, F.Cu at (73.0, 141.2)
- added D_R2C13: Diode, Diode_SMD:D_SOD-123, F.Cu at (84.5, 137.9)
- added D_R2C14: Diode, Diode_SMD:D_SOD-123, F.Cu at (78.8, 137.9)
- added D_R2C15: Diode, Diode_SMD:D_SOD-123, F.Cu at (73.0, 137.9)
- added D_R2C2: Diode, Diode_SMD:D_SOD-123, F.Cu at (84.5, 141.2)
- added D_R2C3: Diode, Diode_SMD:D_SOD-123, F.Cu at (78.8, 144.6)
- added D_R2C4: Diode, Diode_SMD:D_SOD-123, F.Cu at (90.3, 137.9)
- added D_R2C5: Diode, Diode_SMD:D_SOD-123, F.Cu at (73.0, 147.9)
- added D_R2C6: Diode, Diode_SMD:D_SOD-123, F.Cu at (67.3, 147.9)
- added D_R2C7: Diode, Diode_SMD:D_SOD-123, F.Cu at (61.5, 147.9)
- added D_R2C8: Diode, Diode_SMD:D_SOD-123, F.Cu at (73.0, 144.6)
- added D_R2C9: Diode, Diode_SMD:D_SOD-123, F.Cu at (67.3, 144.6)
- added D_R3C0: Diode, Diode_SMD:D_SOD-123, F.Cu at (67.3, 141.2)
- added D_R3C1: Diode, Diode_SMD:D_SOD-123, F.Cu at (61.5, 141.2)
- added D_R3C10: Diode, Diode_SMD:D_SOD-123, F.Cu at (61.5, 137.9)
- added D_R3C11: Diode, Diode_SMD:D_SOD-123, F.Cu at (55.8, 137.9)
- added D_R3C12: Diode, Diode_SMD:D_SOD-123, F.Cu at (50.0, 141.2)
- added D_R3C13: Diode, Diode_SMD:D_SOD-123, F.Cu at (44.3, 141.2)
- added D_R3C14: Diode, Diode_SMD:D_SOD-123, F.Cu at (50.0, 137.9)
- added D_R3C15: Diode, Diode_SMD:D_SOD-123, F.Cu at (44.3, 137.9)
- added D_R3C2: Diode, Diode_SMD:D_SOD-123, F.Cu at (55.8, 147.9)
- added D_R3C3: Diode, Diode_SMD:D_SOD-123, F.Cu at (67.3, 137.9)
- added D_R3C4: Diode, Diode_SMD:D_SOD-123, F.Cu at (50.0, 147.9)
- added D_R3C5: Diode, Diode_SMD:D_SOD-123, F.Cu at (44.3, 147.9)
- added D_R3C6: Diode, Diode_SMD:D_SOD-123, F.Cu at (55.8, 144.6)
- added D_R3C7: Diode, Diode_SMD:D_SOD-123, F.Cu at (50.0, 144.6)
- added D_R3C8: Diode, Diode_SMD:D_SOD-123, F.Cu at (44.3, 144.6)
- added D_R3C9: Diode, Diode_SMD:D_SOD-123, F.Cu at (55.8, 141.2)
- added MX_R0C0_ESC1: MX-NoLED, MX_Alps_Hybrid:MX-1U-NoLED, F.Cu at (51.5, 25.1)
- added MX_R0C10_P1: MX-NoLED, MX_Alps_Hybrid:MX-1U-NoLED, F.Cu at (213.1, 126.1)
- added MX_R0C11_LBRKT1: MX-NoLED, MX_Alps_Hybrid:MX-1U-NoLED, F.Cu at (273.7, 45.3)
- added MX_R0C12_RBRKT1: MX-NoLED, MX_Alps_Hybrid:MX-1U-NoLED, F.Cu at (253.5, 65.5)
- added MX_R0C13_7: MX-NoLED, MX_Alps_Hybrid:MX-1U-NoLED, F.Cu at (233.3, 85.7)
- added MX_R0C14_8: MX-NoLED, MX_Alps_Hybrid:MX-1U-NoLED, F.Cu at (213.1, 105.9)
- added MX_R0C15_9: MX-NoLED, MX_Alps_Hybrid:MX-1U-NoLED, F.Cu at (192.9, 126.1)
- added MX_R0C1_Q1: MX-NoLED, MX_Alps_Hybrid:MX-1U-NoLED, F.Cu at (273.7, 25.1)
- added MX_R0C2_W1: MX-NoLED, MX_Alps_Hybrid:MX-1U-NoLED, F.Cu at (253.5, 45.3)
- added MX_R0C3_E1: MX-NoLED, MX_Alps_Hybrid:MX-1U-NoLED, F.Cu at (233.3, 65.5)
- added MX_R0C4_R1: MX-NoLED, MX_Alps_Hybrid:MX-1U-NoLED, F.Cu at (213.1, 85.7)
- added MX_R0C5_T1: MX-NoLED, MX_Alps_Hybrid:MX-1U-NoLED, F.Cu at (192.9, 105.9)
- added MX_R0C6_Y1: MX-NoLED, MX_Alps_Hybrid:MX-1U-NoLED, F.Cu at (172.7, 126.1)
- added MX_R0C7_U1: MX-NoLED, MX_Alps_Hybrid:MX-1U-NoLED, F.Cu at (253.5, 25.1)
- added MX_R0C8_I1: MX-NoLED, MX_Alps_Hybrid:MX-1U-NoLED, F.Cu at (233.3, 45.3)
- added MX_R0C9_O1: MX-NoLED, MX_Alps_Hybrid:MX-1U-NoLED, F.Cu at (213.1, 65.5)
- added MX_R1C0_TAB1: MX-NoLED, MX_Alps_Hybrid:MX-1U-NoLED, F.Cu at (192.9, 85.7)
- added MX_R1C10_SCLN1: MX-NoLED, MX_Alps_Hybrid:MX-1U-NoLED, F.Cu at (172.7, 105.9)
- added MX_R1C11_SQTE1: MX-NoLED, MX_Alps_Hybrid:MX-1U-NoLED, F.Cu at (152.5, 126.1)
- added MX_R1C12_RTRN1: MX-NoLED, MX_Alps_Hybrid:MX-1U-NoLED, F.Cu at (233.3, 25.1)
- added MX_R1C13_4: MX-NoLED, MX_Alps_Hybrid:MX-1U-NoLED, F.Cu at (213.1, 45.3)
- added MX_R1C14_5: MX-NoLED, MX_Alps_Hybrid:MX-1U-NoLED, F.Cu at (192.9, 65.5)
- added MX_R1C15_6: MX-NoLED, MX_Alps_Hybrid:MX-1U-NoLED, F.Cu at (172.7, 85.7)
- added MX_R1C1_A1: MX-NoLED, MX_Alps_Hybrid:MX-1U-NoLED, F.Cu at (152.5, 105.9)
- added MX_R1C2_S1: MX-NoLED, MX_Alps_Hybrid:MX-1U-NoLED, F.Cu at (132.3, 126.1)
- added MX_R1C3_D1: MX-NoLED, MX_Alps_Hybrid:MX-1U-NoLED, F.Cu at (213.1, 25.1)
- added MX_R1C4_F1: MX-NoLED, MX_Alps_Hybrid:MX-1U-NoLED, F.Cu at (192.9, 45.3)
- added MX_R1C5_G1: MX-NoLED, MX_Alps_Hybrid:MX-1U-NoLED, F.Cu at (172.7, 65.5)
- added MX_R1C6_H1: MX-NoLED, MX_Alps_Hybrid:MX-1U-NoLED, F.Cu at (152.5, 85.7)
- added MX_R1C7_J1: MX-NoLED, MX_Alps_Hybrid:MX-1U-NoLED, F.Cu at (132.3, 105.9)
- added MX_R1C8_K1: MX-NoLED, MX_Alps_Hybrid:MX-1U-NoLED, F.Cu at (112.1, 126.1)
- added MX_R1C9_L1: MX-NoLED, MX_Alps_Hybrid:MX-1U-NoLED, F.Cu at (192.9, 25.1)
- added MX_R2C0_SHIFT1: MX-NoLED, MX_Alps_Hybrid:MX-1U-NoLED, F.Cu at (172.7, 45.3)
- added MX_R2C10_SLSH1: MX-NoLED, MX_Alps_Hybrid:MX-1U-NoLED, F.Cu at (152.5, 65.5)
- added MX_R2C11_BSLSH1: MX-NoLED, MX_Alps_Hybrid:MX-1U-NoLED, F.Cu at (132.3, 85.7)
- added MX_R2C12_UARR1: MX-NoLED, MX_Alps_Hybrid:MX-1U-NoLED, F.Cu at (112.1, 105.9)
- added MX_R2C13_1: MX-NoLED, MX_Alps_Hybrid:MX-1U-NoLED, F.Cu at (91.9, 126.1)
- added MX_R2C14_2: MX-NoLED, MX_Alps_Hybrid:MX-1U-NoLED, F.Cu at (172.7, 25.1)
- added MX_R2C15_3: MX-NoLED, MX_Alps_Hybrid:MX-1U-NoLED, F.Cu at (152.5, 45.3)
- added MX_R2C1_Z1: MX-NoLED, MX_Alps_Hybrid:MX-1U-NoLED, F.Cu at (132.3, 65.5)
- added MX_R2C3_C1: MX-NoLED, MX_Alps_Hybrid:MX-1U-NoLED, F.Cu at (112.1, 85.7)
- added MX_R2C4_V1: MX-NoLED, MX_Alps_Hybrid:MX-1U-NoLED, F.Cu at (91.9, 105.9)
- added MX_R2C5_B1: MX-NoLED, MX_Alps_Hybrid:MX-1U-NoLED, F.Cu at (71.7, 126.1)
- added MX_R2C6_N1: MX-NoLED, MX_Alps_Hybrid:MX-1U-NoLED, F.Cu at (152.5, 25.1)
- added MX_R2C7_M1: MX-NoLED, MX_Alps_Hybrid:MX-1U-NoLED, F.Cu at (132.3, 45.3)
- added MX_R2C8_CMMA1: MX-NoLED, MX_Alps_Hybrid:MX-1U-NoLED, F.Cu at (112.1, 65.5)
- added MX_R2C9_PERI1: MX-NoLED, MX_Alps_Hybrid:MX-1U-NoLED, F.Cu at (91.9, 85.7)
- added MX_R3C0_FN1: MX-NoLED, MX_Alps_Hybrid:MX-1U-NoLED, F.Cu at (71.7, 105.9)
- added MX_R3C10_RSHIFT1: MX-NoLED, MX_Alps_Hybrid:MX-1U-NoLED, F.Cu at (51.5, 126.1)
- added MX_R3C11_LARR1: MX-NoLED, MX_Alps_Hybrid:MX-1U-NoLED, F.Cu at (132.3, 25.1)
- added MX_R3C12_DARR1: MX-NoLED, MX_Alps_Hybrid:MX-1U-NoLED, F.Cu at (112.1, 45.3)
- added MX_R3C13_0: MX-NoLED, MX_Alps_Hybrid:MX-1U-NoLED, F.Cu at (91.9, 65.5)
- added MX_R3C13_RARR1: MX-NoLED, MX_Alps_Hybrid:MX-1U-NoLED, F.Cu at (71.7, 85.7)
- added MX_R3C15_BKSPC1: MX-NoLED, MX_Alps_Hybrid:MX-1U-NoLED, F.Cu at (51.5, 105.9)
- added MX_R3C1_CTRLL1: MX-NoLED, MX_Alps_Hybrid:MX-1U-NoLED, F.Cu at (112.1, 25.1)
- added MX_R3C2_ALTL1: MX-NoLED, MX_Alps_Hybrid:MX-1U-NoLED, F.Cu at (91.9, 45.3)
- added MX_R3C2_X1: MX-NoLED, MX_Alps_Hybrid:MX-1U-NoLED, F.Cu at (71.7, 65.5)
- added MX_R3C3_CMDL1: MX-NoLED, MX_Alps_Hybrid:MX-1U-NoLED, F.Cu at (51.5, 85.7)
- added MX_R3C4_LAYRD1: MX-NoLED, MX_Alps_Hybrid:MX-1U-NoLED, F.Cu at (91.9, 25.1)
- added MX_R3C5_SPCEL1: MX-NoLED, MX_Alps_Hybrid:MX-1U-NoLED, F.Cu at (71.7, 45.3)
- added MX_R3C6_SPCER1: MX-NoLED, MX_Alps_Hybrid:MX-1U-NoLED, F.Cu at (51.5, 65.5)
- added MX_R3C7_LYERU1: MX-NoLED, MX_Alps_Hybrid:MX-1U-NoLED, F.Cu at (71.7, 25.1)
- added MX_R3C8_CMDR1: MX-NoLED, MX_Alps_Hybrid:MX-1U-NoLED, F.Cu at (51.5, 45.3)
- added MX_R3C9_ALTR1: MX-NoLED, MX_Alps_Hybrid:MX-1U-NoLED, F.Cu at (233.3, 105.9)
- moved C1 79.9 mm to (48.9, 170.0)
- moved C3 79.9 mm to (54.1, 176.1)
- moved C5 79.9 mm to (37.7, 170.9)
- moved C6 79.9 mm to (35.9, 179.7)
- moved C7 79.9 mm to (49.4, 190.6)
- moved F1 79.9 mm to (20.0, 175.8)
- moved R1 79.9 mm to (22.8, 166.1)
- moved R3 79.9 mm to (25.9, 166.1)
- moved R4 79.9 mm to (54.1, 186.2)
- moved SW1 79.9 mm to (20.7, 188.7)
- moved Y1 79.9 mm to (45.5, 170.0)
- moved C2 79.9 mm to (41.9, 169.9)
- moved C4 79.9 mm to (36.1, 186.6)
- moved R2 79.9 mm to (33.1, 172.2)
- moved U1 79.9 mm to (45.4, 181.1)
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Connections:
- U1 pad 12: Net-(U1-Pad12) -> COL3
- U1 pad 18: Net-(U1-Pad18) -> COL6
- U1 pad 19: Net-(U1-Pad19) -> COL7
- U1 pad 20: Net-(U1-Pad20) -> COL8
- U1 pad 21: Net-(U1-Pad21) -> COL9
- U1 pad 22: Net-(U1-Pad22) -> COL11
- U1 pad 25: Net-(U1-Pad25) -> COL10
- U1 pad 26: Net-(U1-Pad26) -> COL12
- U1 pad 27: ROW0 -> COL13
- U1 pad 28: COL1 -> COL0
- U1 pad 29: COL0 -> COL1
- U1 pad 30: ROW1 -> COL2
- U1 pad 31: Net-(U1-Pad31) -> COL4
- U1 pad 32: Net-(U1-Pad32) -> COL5
- U1 pad 36: Net-(U1-Pad36) -> ROW3
- U1 pad 37: Net-(U1-Pad37) -> ROW2
- U1 pad 38: Net-(U1-Pad38) -> ROW1
- U1 pad 39: Net-(U1-Pad39) -> ROW0
- U1 pad 40: Net-(U1-Pad40) -> COL15
- U1 pad 41: Net-(U1-Pad41) -> COL14
Routing:
- net COL13: track 0.00 -> 49.6 mm
- net ROW0: track 49.6 -> 0.00 mm
- net ROW1: track 47.3 -> 0.00 mm
- net COL2: track 0.00 -> 47.3 mm
- net COL1: track 54.5 -> 10.6 mm
- net COL0: track 29.6 -> 54.5 mm
- net (no net): track 0.00 -> 19.1 mm

Commit message: I just wired up a 63-key board. yiiikes.
Parts:
- removed C1, C2: 22pF, Capacitor_SMD:C_0805_2012Metric
- removed C3, C4, C5: 0.1uF, Capacitor_SMD:C_0805_2012Metric
- removed C6: 1uF, Capacitor_SMD:C_0805_2012Metric
- removed C7: 10uF, Capacitor_SMD:C_0805_2012Metric
- removed F1: 500mA, Fuse:Fuse_1206_3216Metric
- removed MX_R0C15_9, MX_R1C15_6, MX_R2C15_3, MX_R3C13_0, MX_R3C15_BKSPC1, MX_R3C2_X1: MX-NoLED, MX_Alps_Hybrid:MX-1U-NoLED
- removed R1, R3: 22, Resistor_SMD:R_0805_2012Metric
- removed R2, R4: 10k, Resistor_SMD:R_0805_2012Metric
- removed SW1: SW_Push, random-keyboard-parts:SKQG-1155865
- added C_D0: 0.1uF, Capacitor_SMD:C_0805_2012Metric, B.Cu at (-3.94, 63.0)
- added C_D1: 0.1uF, Capacitor_SMD:C_0805_2012Metric, B.Cu at (-8.76, 77.5)
- added C_D2: 0.1uF, Capacitor_SMD:C_0805_2012Metric, B.Cu at (-20.6, 57.8)
- added C_D3: 10uF, Capacitor_SMD:C_0805_2012Metric, B.Cu at (-22.0, 73.4)
- added C_UCAP1: 1uF, Capacitor_SMD:C_0805_2012Metric, B.Cu at (-21.5, 65.8)
- added C_XTAL0: 22pF, Capacitor_SMD:C_0805_2012Metric, B.Cu at (-8.64, 56.8)
- added C_XTAL1: 22pF, Capacitor_SMD:C_0805_2012Metric, B.Cu at (-16.4, 56.8)
- added F_VBUS1: 500mA, Fuse:Fuse_1206_3216Metric, B.Cu at (-35.8, 65.3)
- added MX_R0C15_BKSPC1: MX-NoLED, MX_Alps_Hybrid:MX-1U-NoLED, F.Cu at (246.5, 8.26)
- added MX_R1C15_9: MX-NoLED, MX_Alps_Hybrid:MX-1U-NoLED, F.Cu at (332.1, 27.3)
- added MX_R2C15_6: MX-NoLED, MX_Alps_Hybrid:MX-1U-NoLED, F.Cu at (332.1, 46.4)
- added MX_R2C2_X1: MX-NoLED, MX_Alps_Hybrid:MX-1U-NoLED, F.Cu at (65.4, 65.4)
- added MX_R3C14_0: MX-NoLED, MX_Alps_Hybrid:MX-1U-NoLED, F.Cu at (322.6, 84.6)
- added MX_R3C15_1: MX-NoLED, MX_Alps_Hybrid:MX-1U-NoLED, F.Cu at (332.1, 65.4)
- added R_D+1: 22, Resistor_SMD:R_0805_2012Metric, B.Cu at (-32.6, 53.3)
- added R_D-1: 22, Resistor_SMD:R_0805_2012Metric, B.Cu at (-34.8, 53.3)
- added R_HWB1: 10k, Resistor_SMD:R_0805_2012Metric, B.Cu at (-3.94, 73.0)
- added R_RESET1: 10k, Resistor_SMD:R_0805_2012Metric, B.Cu at (-25.0, 57.8)
- added SW_PUSH_RESET1: SW_Push, random-keyboard-parts:SKQG-1155865, B.Cu at (-35.7, 80.6)
- D_R0C0, D_R0C1, D_R0C10, D_R0C11, D_R0C12, D_R0C13, D_R0C14, D_R0C15, D_R0C2, D_R0C3, D_R0C4, D_R0C5, D_R0C6, D_R0C7, D_R0C8, D_R0C9, D_R1C0, D_R1C1, D_R1C10, D_R1C11, D_R1C12, D_R1C13, D_R1C14, D_R1C15, D_R1C2, D_R1C3, D_R1C4, D_R1C5, D_R1C6, D_R1C7, D_R1C8, D_R1C9, D_R2C0, D_R2C1, D_R2C10, D_R2C11, D_R2C12, D_R2C13, D_R2C14, D_R2C15, D_R2C2, D_R2C3, D_R2C4, D_R2C5, D_R2C6, D_R2C7, D_R2C8, D_R2C9, D_R3C0, D_R3C1, D_R3C10, D_R3C11, D_R3C12, D_R3C13, D_R3C14, D_R3C15, D_R3C2, D_R3C3, D_R3C4, D_R3C5, D_R3C6, D_R3C7, D_R3C8, D_R3C9: moved to B.Cu
- moved D_R3C15 305.0 mm to (340.4, 64.8), turned to 90 degrees
- moved D_R3C14 286.0 mm to (330.8, 83.8), turned to 90 degrees
- moved D_R2C15 282.8 mm to (340.4, 45.7), turned to 90 degrees
- moved D_R1C15 275.1 mm to (340.4, 26.7), turned to 90 degrees
- moved D_R2C14 253.3 mm to (321.3, 64.8), turned to 90 degrees
- moved D_R3C13 253.0 mm to (292.7, 93.3), turned to 90 degrees
- moved D_R0C14 249.2 mm to (321.3, 26.7), turned to 90 degrees
- moved D_R1C14 243.4 mm to (321.3, 45.7), turned to 90 degrees
- moved D_R2C13 229.7 mm to (302.3, 64.8), turned to 90 degrees
- moved D_R3C12 228.7 mm to (273.7, 93.3), turned to 90 degrees
- moved D_R0C13 227.7 mm to (302.3, 26.7), turned to 90 degrees
- moved MX_R0C1_Q1 227.4 mm to (46.4, 27.3)
- moved D_R1C13 220.7 mm to (302.3, 45.7), turned to 90 degrees
- moved MX_R3C13_RARR1 212.9 mm to (284.5, 94.0)
- moved D_R2C12 212.3 mm to (274.3, 73.7), turned to 90 degrees
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Connections:
- U1 pad 11: Net-(U1-Pad11) -> COL15
- U1 pad 12: COL3 -> Net-(U1-Pad12)
- U1 pad 18: COL6 -> COL14
- U1 pad 19: COL7 -> COL13
- U1 pad 20: COL8 -> COL12
- U1 pad 21: COL9 -> COL11
- U1 pad 22: COL11 -> COL10
- U1 pad 25: COL10 -> COL9
- U1 pad 26: COL12 -> COL8
- U1 pad 27: COL13 -> COL7
- U1 pad 28: COL0 -> COL6
- U1 pad 29: COL1 -> COL5
- U1 pad 30: COL2 -> COL4
- U1 pad 31: COL4 -> COL3
- U1 pad 32: COL5 -> COL2
- U1 pad 36: ROW3 -> COL1
- U1 pad 37: ROW2 -> COL0
- U1 pad 38: ROW1 -> ROW0
- U1 pad 39: ROW0 -> ROW1
- U1 pad 40: COL15 -> ROW2
- U1 pad 41: COL14 -> ROW3
Routing:
- net COL9: track 0.00 -> 525.6 mm
- net ROW0: track 0.00 -> 473.2 mm
- net COL15: track 0.00 -> 466.1 mm
- net COL14: track 0.00 -> 430.8 mm
- net ROW1: track 0.00 -> 401.2 mm
- net ROW3: track 0.00 -> 399.1 mm
- net ROW2: track 0.00 -> 396.2 mm
- net COL12: track 0.00 -> 380.7 mm
- net COL13: track 49.6 -> 420.4 mm
- net COL11: track 0.00 -> 360.5 mm
- net COL10: track 0.00 -> 326.9 mm
- net COL8: track 0.00 -> 290.9 mm
- net COL7: track 0.00 -> 271.8 mm
- net COL6: track 0.00 -> 252.7 mm
- net COL5: track 0.00 -> 235.9 mm
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- removed copper zone on B.Cu, net GND

Commit message: wired up switches to ATMega
Parts:
- moved C_D0 202.4 mm to (144.0, 201.2)
- moved C_D2 202.4 mm to (127.4, 196.0)
- moved C_XTAL0 202.4 mm to (139.3, 195.0)
- moved D_R2C12 202.4 mm to (422.3, 211.8)
- moved D_R3C0 202.4 mm to (183.5, 222.0)
- moved D_R3C1 202.4 mm to (202.6, 222.0)
- moved D_R3C10 202.4 mm to (374.0, 222.0)
- moved D_R3C14 202.4 mm to (478.8, 222.0)
- moved D_R3C2 202.4 mm to (221.5, 222.0)
- moved D_R3C3 202.4 mm to (240.7, 222.0)
- moved D_R3C4 202.4 mm to (259.7, 222.0)
- moved D_R3C5 202.4 mm to (278.8, 222.0)
- moved D_R3C6 202.4 mm to (297.7, 222.0)
- moved D_R3C7 202.4 mm to (316.9, 222.0)
- moved D_R3C8 202.4 mm to (335.9, 222.0)
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Other:
- board outline added: 404.8 x 127 mm

Commit message: a few extra tweeks including silkscreen color and adding ground fill
Parts:
- MX_R0C15_BKSPC1, MX_R3C14_0: value MX-NoLED -> MX-2U-NoLED; footprint MX_Alps_Hybrid:MX-1U-NoLED -> MX_Alps_Hybrid:MX-2U-NoLED
Routing:
- added copper zone on B.Cu, net (none)
- added copper zone on B.Cu, net GND
Other:
- board text added: "Keybored v0.1"

Commit message: Fixed up some missed connections
Routing:
- net COL9: track 525.6 -> 462.1 mm
- net GND: track 136.3 -> 150.1 mm
- net +5V: track 100.5 -> 102.8 mm, vias 4 -> 5
- net COL13: track 420.4 -> 422.6 mm
- net COL14: track 430.8 -> 433.0 mm
- net ROW3: track 399.1 -> 399.9 mm
- net COL15: track 466.1 -> 466.9 mm
- removed copper zone on B.Cu, net (none)
