File: keybored.kicad_pcb (KiCad board)
At the start: 2 copper layers, 404.8 x 127 mm, 144 parts, among them U1 ATmega32U4-AU, Y1 16MHz

Commit message: moved MCU above ortho48 section
Parts:
- moved C_XTAL0 114.7 mm to (235.2, 132.1)
- moved Y1 114.7 mm to (231.3, 132.1)
- moved C_D0 114.7 mm to (239.9, 138.3)
- moved C_D1 114.7 mm to (235.1, 152.8)
- moved C_D2 114.7 mm to (223.3, 133.1)
- moved C_XTAL1 114.7 mm to (227.5, 132.1)
- moved R_HWB1 114.7 mm to (239.9, 148.3)
- moved R_RESET1 114.7 mm to (218.8, 133.1)
- moved U1 114.7 mm to (231.2, 143.3)
- moved C_D3 114.7 mm to (221.9, 148.7)
- moved C_UCAP1 114.7 mm to (222.4, 141.1)
- moved F_VBUS1 112.4 mm to (200.0, 133.3)
- moved SW_PUSH_RESET1 110.7 mm to (194.7, 144.9)
- moved R_D-1 108.7 mm to (208.0, 138.4)
- moved R_D+1 108.7 mm to (210.2, 138.4)
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Connections:
- U1 pad 11: COL15 -> Net-(U1-Pad11)
- U1 pad 12: Net-(U1-Pad12) -> ROW3
- U1 pad 18: COL14 -> ROW2
- U1 pad 19: COL13 -> ROW1
- U1 pad 20: COL12 -> ROW0
- U1 pad 21: COL11 -> COL15
- U1 pad 22: COL10 -> COL14
- U1 pad 25: COL9 -> COL13
- U1 pad 26: COL8 -> COL12
- U1 pad 27: COL7 -> COL11
- U1 pad 28: COL6 -> COL10
- U1 pad 29: COL5 -> COL9
- U1 pad 30: COL4 -> COL8
- U1 pad 31: COL3 -> COL7
- U1 pad 32: COL2 -> COL6
- U1 pad 36: COL1 -> COL5
- U1 pad 37: COL0 -> COL4
- U1 pad 38: ROW0 -> COL3
- U1 pad 39: ROW1 -> COL2
- U1 pad 40: ROW2 -> COL1
- U1 pad 41: ROW3 -> COL0
Routing:
- net ROW3: track 399.9 -> 708.3 mm
- net COL9: track 462.1 -> 168.2 mm
- net ROW2: track 396.2 -> 651.7 mm
- net ROW1: track 401.2 -> 624.4 mm
- net COL15: track 466.9 -> 301.7 mm
- net COL7: track 271.8 -> 127.3 mm
- net COL6: track 252.7 -> 110.3 mm
- net COL13: track 422.6 -> 282.2 mm
- net COL5: track 235.9 -> 96.6 mm
- net COL8: track 290.9 -> 151.6 mm
- net COL11: track 360.5 -> 221.4 mm
- net COL10: track 326.9 -> 188.3 mm
- net COL12: track 380.7 -> 242.6 mm
- net COL4: track 214.5 -> 78.4 mm
- net COL14: track 433.0 -> 298.2 mm
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Other:
- board size 404.8 x 127 mm -> 341.3 x 127 mm
- board text removed: "KeyBored"

Commit message: forgot fill zones
Routing:
- net COL15: track 301.7 -> 299.0 mm
- net COL7: track 127.3 -> 129.4 mm
- net COL14: track 298.2 -> 296.4 mm
